Commit message: working on urdf

File: ur3robot/ros_code/urdf/robot.urdf (robot description, URDF)
Before this commit: robot ur3`, 3 links, 1 joints
Links:
- removed link webcam

Commit message: working on video stuff

File: ur3robot/ros_code/urdf/robot.urdf (robot description, URDF)
Before this commit: robot ur3`, 2 links, 1 joints
Links:
- added link webcam
Joints:
- added joint base_link_to_webcam: type fixed, parent base_link, child webcam, origin xyz=0.21 0.051 0.27 rpy=0.0 0.0 0, axis 0 0 0

Commit message: updating urdf

File: ur3robot/ros_code/urdf/robot.urdf (robot description, URDF)
Before this commit: robot ur3`, 3 links, 2 joints
Joints:
- joint base_link_to_laser: origin xyz=0 0 0.3429 rpy=0.0 0.0 3.141592 -> xyz=0 0 0.3429 rpy=0.0 0.0 4.712389
- joint base_link_to_webcam: origin xyz=0.21 0.051 0.27 rpy=0.0 0.0 0 -> xyz=0.21 -0.051 0.27 rpy=0.0 0.0 0

Commit message: added laser filter code

File: ur3robot/ros_code/urdf/robot.urdf (robot description, URDF)
Before this commit: robot ur3`, 3 links, 2 joints
Joints:
- joint base_link_to_laser: origin xyz=0 0 0.3429 rpy=0.0 0.0 4.712389 -> xyz=0 0 0.3429 rpy=0.0 0.0 1.570796

Commit message: updated robot.urdf for imu

File: ur3robot/ros_code/urdf/robot.urdf (robot description, URDF)
Before this commit: robot ur3`, 3 links, 2 joints
Links:
- added link imu
Joints:
- added joint base_link_to_imu: type fixed, parent base_link, child imu, origin xyz=0.198 -0.153 0.458 rpy=0.0 0.0 1.5708, axis 0 0 0

Commit message: updated urdf

File: ur3robot/ros_code/urdf/robot.urdf (robot description, URDF)
Before this commit: robot ur3`, 4 links, 3 joints
Joints:
- joint base_link_to_imu: origin xyz=0.198 -0.153 0.458 rpy=0.0 0.0 1.5708 -> xyz=-0.198 -0.153 0.458 rpy=0.0 0.0 0

Commit message: fixed urdf and working on ekf

File: ur3robot/ros_code/urdf/robot.urdf (robot description, URDF)
Before this commit: robot ur3`, 4 links, 3 joints
Joints:
- joint base_link_to_imu: origin xyz=-0.198 -0.153 0.458 rpy=0.0 0.0 0 -> xyz=-0.198 -0.153 0.458 rpy=0.0 0.0 3.14159

Commit message: updated urdf and freenect.launch

File: ur3robot/ros_code/urdf/robot.urdf (robot description, URDF)
Before this commit: robot ur3`, 4 links, 3 joints
Links:
- added link camera_link
Joints:
- added joint base_link_to_camera_link: type fixed, parent base_link, child camera_link, origin xyz=0 0 0.458 rpy=0.0 0.0 0.0, axis 0 0 0

Commit message: updated urdf, and added tf to kinect_aux

File: ur3robot/ros_code/urdf/robot.urdf (robot description, URDF)
Before this commit: robot ur3`, 5 links, 4 joints
Links:
- added link kinect_base
- added link kinect_pivot
- added link kinect_rotator
Joints:
- removed joint base_link_to_camera_link
- added joint base_link_to_kinect_rotator: type fixed, parent base_link, child kinect_rotator, origin xyz=0.1 0.060 1.19 rpy=0.0 0.0 0.0, axis 0 0 0
- added joint kinect_pivot_to_camera_link: type fixed, parent kinect_pivot, child camera_link, origin xyz=0.0272 0.0117 0.034 rpy=0.0 0.0 0.0, axis 0 0 0
- added joint kinect_rotator_to_kinect_base: type fixed, parent kinect_rotator, child kinect_base, origin xyz=0.0067 0 0.0169 rpy=0.0 0.0 0.0, axis 0 0 0

Commit message: Update robot.urdf

File: ur3robot/ros_code/urdf/robot.urdf (robot description, URDF)
Before this commit: robot ur3`, 8 links, 6 joints
Joints:
- removed joint kinect_pivot_to_camera_link

Commit message: Update robot.urdf

File: ur3robot/ros_code/urdf/robot.urdf (robot description, URDF)
Before this commit: robot ur3, 8 links, 5 joints
Links:
- removed link camera_link
- removed link kinect_pivot

Commit message: working on stuff

File: ur3robot/ros_code/urdf/robot.urdf (robot description, URDF)
Before this commit: robot ur3, 6 links, 5 joints
Joints:
- joint kinect_rotator_to_kinect_base: origin xyz=0.0067 0 0.0169 rpy=0.0 0.0 0.0 -> xyz=0.0102 0 0.0306 rpy=0.0 0.0 0.0

Commit message: Added all kinect tf to my robot urdf, so now I will have to rewrite kinect_aux to publish joint state

File: ur3robot/ros_code/urdf/robot.urdf (robot description, URDF)
Before this commit: robot ur3, 6 links, 5 joints
Links:
- added link camera_depth_frame
- added link camera_depth_optical_frame
- added link camera_link
- added link camera_rgb_frame
- added link camera_rgb_optical_frame
- added link tower
Joints:
- added joint base_link_to_tower: type revolute, parent base_link, child tower, origin xyz=0.1 0.060 0.513 rpy=0.0 0.0 0.0, axis 0 0 1
- added joint camera_depth_frame_to_camera_depth_optical_frame: type fixed, parent camera_depth_frame, child camera_depth_optical_frame, origin xyz=0 0 0 rpy=$(arg optical_rotate), axis 0 0 0
- added joint camera_link_to_camera_depth_frame: type fixed, parent camera_link, child camera_depth_frame, origin xyz=0 -0.02 0 rpy=0.0 0.0 0.0, axis 0 0 0
- added joint camera_link_to_camera_rgb_frame: type fixed, parent camera_link, child camera_rgb_frame, origin xyz=0 -0.045 0 rpy=0.0 0.0 0.0, axis 0 0 0
- added joint camera_rgb_frame_to_camera_rgb_optical_frame: type fixed, parent camera_rgb_frame, child camera_rgb_optical_frame, origin xyz=0 0 0 rpy=$(arg optical_rotate), axis 0 0 0
- added joint kinect_base_to_camera_link: type revolute, parent kinect_base, child camera_link, origin xyz=0.0067 0.0117 0.0169 rpy=0.0 0.0 0.0, axis 0 1 0
- added joint tower_to_kinect_rotator: type fixed, parent tower, child kinect_rotator, origin xyz=0 0.0 0.677 rpy=0.0 0.0 0.0, axis 0 0 0
- joint kinect_rotator_to_kinect_base: axis 0 0 0 -> 0 0 1; type fixed -> revolute

Commit message: added limits to urdf

File: ur3robot/ros_code/urdf/robot.urdf (robot description, URDF)
Before this commit: robot ur3, 12 links, 12 joints
Joints:
- joint base_link_to_tower: limit (none) -> lower=-3.14159 upper=3.14159 effort=10 velocity=1.0
- joint kinect_base_to_camera_link: limit (none) -> lower=-0.7679449 upper=0.3141593 effort=5 velocity=0.5
- joint kinect_rotator_to_kinect_base: limit (none) -> lower=-3.14159 upper=3.14159 effort=10 velocity=1.0

Commit message: Update robot.urdf

File: ur3robot/ros_code/urdf/robot.urdf (robot description, URDF)
Before this commit: robot ur3, 12 links, 12 joints
Joints:
- joint camera_depth_frame_to_camera_depth_optical_frame: origin xyz=0 0 0 rpy=$(arg optical_rotate) -> xyz=0 0 0 rpy=-1.5707963267948966 0 -1.5707963267948966
- joint camera_rgb_frame_to_camera_rgb_optical_frame: origin xyz=0 0 0 rpy=$(arg optical_rotate) -> xyz=0 0 0 rpy=-1.5707963267948966 0 -1.5707963267948966

Commit message: maybe found issue in urdf

File: ur3robot/ros_code/urdf/robot.urdf (robot description, URDF)
Before this commit: robot ur3, 12 links, 12 joints
Joints:
- removed joint base_link_to_kinect_rotator

Commit message: trying to go back to old tf to see if that fixes the warning problem

File: ur3robot/ros_code/urdf/robot.urdf (robot description, URDF)
Before this commit: robot ur3, 12 links, 11 joints
Links:
- removed link camera_depth_frame
- removed link camera_depth_optical_frame
- removed link camera_link
- removed link camera_rgb_frame
- removed link camera_rgb_optical_frame
Joints:
- removed joint camera_depth_frame_to_camera_depth_optical_frame
- removed joint camera_link_to_camera_depth_frame
- removed joint camera_link_to_camera_rgb_frame
- removed joint camera_rgb_frame_to_camera_rgb_optical_frame
- removed joint kinect_base_to_camera_link

Commit message: Update robot.urdf

File: ur3robot/ros_code/urdf/robot.urdf (robot description, URDF)
Before this commit: robot ur3, 7 links, 6 joints
Joints:
- joint base_link_to_tower: type revolute -> fixed
- joint kinect_rotator_to_kinect_base: type revolute -> fixed

Commit message: Update robot.urdf

File: ur3robot/ros_code/urdf/robot.urdf (robot description, URDF)
Before this commit: robot ur3, 7 links, 6 joints
Joints:
- joint base_link_to_tower: type fixed -> revolute

Commit message: Update robot.urdf

File: ur3robot/ros_code/urdf/robot.urdf (robot description, URDF)
Before this commit: robot ur3, 7 links, 6 joints
Joints:
- joint base_link_to_tower: limit lower=-3.14159 upper=3.14159 effort=10 velocity=1.0 -> (none); type revolute -> continuous

Commit message: working on joints

File: ur3robot/ros_code/urdf/robot.urdf (robot description, URDF)
Before this commit: robot ur3, 7 links, 6 joints
Joints:
- added joint kinect_base_to_camera_link: type revolute, parent kinect_base, child camera_link, origin xyz=0.0067 0.0117 0.0169 rpy=0.0 0.0 0.0, axis 0 1 0, limit lower=-0.7679449 upper=0.3141593 effort=5 velocity=0.5
- joint base_link_to_tower: type continuous -> fixed

Commit message: Update robot.urdf

File: ur3robot/ros_code/urdf/robot.urdf (robot description, URDF)
Before this commit: robot ur3, 7 links, 7 joints
Links:
- added link camera_link

Commit message: Finally figured out that my erroring was due to too low publish speed from joint state

File: ur3robot/ros_code/urdf/robot.urdf (robot description, URDF)
Before this commit: robot ur3, 8 links, 7 joints
Links:
- added link camera_depth_frame
- added link camera_depth_optical_frame
- added link camera_rgb_frame
- added link camera_rgb_optical_frame
Joints:
- added joint camera_depth_frame_to_camera_depth_optical_frame: type fixed, parent camera_depth_frame, child camera_depth_optical_frame, origin xyz=0 0 0 rpy=-1.5707963267948966 0 -1.5707963267948966, axis 0 0 0
- added joint camera_link_to_camera_depth_frame: type fixed, parent camera_link, child camera_depth_frame, origin xyz=0 -0.02 0 rpy=0.0 0.0 0.0, axis 0 0 0
- added joint camera_link_to_camera_rgb_frame: type fixed, parent camera_link, child camera_rgb_frame, origin xyz=0 -0.045 0 rpy=0.0 0.0 0.0, axis 0 0 0
- added joint camera_rgb_frame_to_camera_rgb_optical_frame: type fixed, parent camera_rgb_frame, child camera_rgb_optical_frame, origin xyz=0 0 0 rpy=-1.5707963267948966 0 -1.5707963267948966, axis 0 0 0
- joint base_link_to_tower: type fixed -> revolute
- joint kinect_rotator_to_kinect_base: type fixed -> revolute

Commit message: fixed bug

File: ur3robot/ros_code/urdf/robot.urdf (robot description, URDF)
Before this commit: robot ur3, 12 links, 11 joints
Joints:
- joint base_link_to_tower: limit (none) -> lower=-3.14159 upper=3.14159 effort=10 velocity=1.0

Commit message: updated scara code and urdf

File: ur3robot/ros_code/urdf/robot.urdf (robot description, URDF)
Before this commit: robot ur3, 12 links, 11 joints
Links:
- added link scara_arm_base
- added link scara_arm_gripper
- added link scara_arm_joint
Joints:
- added joint scara_arm_base_to_scara_arm_joint: type revolute, parent scara_arm_base, child scara_arm_joint, origin xyz=0.3 0 0 rpy=0.0 0.0 0.0, axis 0 0 1, limit lower=-3 upper=3 effort=10 velocity=1.0
- added joint scara_arm_joint_to_scara_arm_gripper: type fixed, parent scara_arm_joint, child scara_arm_gripper, origin xyz=0.3 0 0 rpy=0.0 0.0 0.0, axis 0 0 0
- added joint tower_to_scara_arm_base: type prismatic, parent tower, child scara_arm_base, origin xyz=0 0 0 rpy=0.0 0.0 0.0, axis 0 0 1, limit lower=0 upper=0.677 effort=10 velocity=1.0

Commit message: updated urdf

File: ur3robot/ros_code/urdf/robot.urdf (robot description, URDF)
Before this commit: robot ur3, 15 links, 14 joints
Links:
- removed link camera_link
- removed link kinect_base
- added link kinect_pivot
Joints:
- removed joint camera_link_to_camera_depth_frame
- removed joint camera_link_to_camera_rgb_frame
- removed joint kinect_base_to_camera_link
- removed joint kinect_rotator_to_kinect_base
- added joint camera_depth_frame_to_camera_rgb_frame: type fixed, parent camera_depth_frame, child camera_rgb_frame, origin xyz=0 -0.026 0 rpy=0.0 0.0 0.0, axis 0 0 0
- added joint kinect_pivot_to_camera_depth_frame: type revolute, parent kinect_pivot, child camera_depth_frame, origin xyz=0.029 0.011 0.034 rpy=0.0 0.0 0.0, axis 0 1 0, limit lower=-0.7679449 upper=0.3141593 effort=5 velocity=0.5
- added joint kinect_rotator_to_kinect_pivot: type revolute, parent kinect_rotator, child kinect_pivot, origin xyz=0.0106 0 0.0307 rpy=0.0 0.0 0.0, axis 0 0 1, limit lower=-3.14159 upper=3.14159 effort=10 velocity=1.0
- joint base_link_to_tower: origin xyz=0.1 0.060 0.513 rpy=0.0 0.0 0.0 -> xyz=0.1 0.060 0.5 rpy=0.0 0.0 0.0
- joint tower_to_kinect_rotator: origin xyz=0 0.0 0.677 rpy=0.0 0.0 0.0 -> xyz=0 0.0 0.691 rpy=0.0 0.0 0.0
