Commit message: fixed location of meshes

File: ur3robot/ros_code/urdf/ur3.xacro (robot description, xacro)
@@ -5,5 +5,5 @@
     <origin xyz="0 0 0" rpy="0 0 0"/>
     <geometry>
-      <mesh filename="package://ur3_description/meshes/base_link.stl" scale="0.001 0.001 0.001"/>
+      <mesh filename="package://ur3robot/meshes/base_link.stl" scale="0.001 0.001 0.001"/>
     </geometry>
     <material name="silver_default"/>
@@ -12,5 +12,5 @@
     <origin xyz="0 0 0" rpy="0 0 0"/>
     <geometry>
-      <mesh filename="package://ur3_description/meshes/base_link.stl" scale="0.001 0.001 0.001"/>
+      <mesh filename="package://ur3robot/meshes/base_link.stl" scale="0.001 0.001 0.001"/>
     </geometry>
   </collision>
@@ -20,5 +20,5 @@
     <origin xyz="-0.105418 -0.06341 -0.487908" rpy="0 0 0"/>
     <geometry>
-      <mesh filename="package://ur3_description/meshes/tower.stl" scale="0.001 0.001 0.001"/>
+      <mesh filename="package://ur3robot/meshes/tower.stl" scale="0.001 0.001 0.001"/>
     </geometry>
     <material name="silver_default"/>
@@ -27,5 +27,5 @@
     <origin xyz="-0.105418 -0.06341 -0.487908" rpy="0 0 0"/>
     <geometry>
-      <mesh filename="package://ur3_description/meshes/tower.stl" scale="0.001 0.001 0.001"/>
+      <mesh filename="package://ur3robot/meshes/tower.stl" scale="0.001 0.001 0.001"/>
     </geometry>
   </collision>
@@ -35,5 +35,5 @@
     <origin xyz="-0.143418 -0.06341 -0.829408" rpy="0 0 0"/>
     <geometry>
-      <mesh filename="package://ur3_description/meshes/arm1.stl" scale="0.001 0.001 0.001"/>
+      <mesh filename="package://ur3robot/meshes/arm1.stl" scale="0.001 0.001 0.001"/>
     </geometry>
     <material name="silver_default"/>
@@ -42,5 +42,5 @@
     <origin xyz="-0.143418 -0.06341 -0.829408" rpy="0 0 0"/>
     <geometry>
-      <mesh filename="package://ur3_description/meshes/arm1.stl" scale="0.001 0.001 0.001"/>
+      <mesh filename="package://ur3robot/meshes/arm1.stl" scale="0.001 0.001 0.001"/>
     </geometry>
   </collision>
@@ -50,5 +50,5 @@
     <origin xyz="-0.331194 -0.06341 -0.872808" rpy="0 0 0"/>
     <geometry>
-      <mesh filename="package://ur3_description/meshes/arm2.stl" scale="0.001 0.001 0.001"/>
+      <mesh filename="package://ur3robot/meshes/arm2.stl" scale="0.001 0.001 0.001"/>
     </geometry>
     <material name="silver_default"/>
@@ -57,5 +57,5 @@
     <origin xyz="-0.331194 -0.06341 -0.872808" rpy="0 0 0"/>
     <geometry>
-      <mesh filename="package://ur3_description/meshes/arm2.stl" scale="0.001 0.001 0.001"/>
+      <mesh filename="package://ur3robot/meshes/arm2.stl" scale="0.001 0.001 0.001"/>
     </geometry>
   </collision>

Commit message: Testing

File: ur3robot/ros_code/urdf/ur3.xacro (robot description, xacro)
@@ -5,5 +5,5 @@
     <origin xyz="0 0 0" rpy="0 0 0"/>
     <geometry>
-      <mesh filename="package://ur3robot/meshes/base_link.stl" scale="0.001 0.001 0.001"/>
+      <mesh filename="package://ur3master/meshes/base_link.stl" scale="0.001 0.001 0.001"/>
     </geometry>
     <material name="silver_default"/>
@@ -12,5 +12,5 @@
     <origin xyz="0 0 0" rpy="0 0 0"/>
     <geometry>
-      <mesh filename="package://ur3robot/meshes/base_link.stl" scale="0.001 0.001 0.001"/>
+      <mesh filename="package://ur3master/meshes/base_link.stl" scale="0.001 0.001 0.001"/>
     </geometry>
   </collision>
@@ -20,5 +20,5 @@
     <origin xyz="-0.105418 -0.06341 -0.487908" rpy="0 0 0"/>
     <geometry>
-      <mesh filename="package://ur3robot/meshes/tower.stl" scale="0.001 0.001 0.001"/>
+      <mesh filename="package://ur3master/meshes/tower.stl" scale="0.001 0.001 0.001"/>
     </geometry>
     <material name="silver_default"/>
@@ -27,5 +27,5 @@
     <origin xyz="-0.105418 -0.06341 -0.487908" rpy="0 0 0"/>
     <geometry>
-      <mesh filename="package://ur3robot/meshes/tower.stl" scale="0.001 0.001 0.001"/>
+      <mesh filename="package://ur3master/meshes/tower.stl" scale="0.001 0.001 0.001"/>
     </geometry>
   </collision>
@@ -35,5 +35,5 @@
     <origin xyz="-0.143418 -0.06341 -0.829408" rpy="0 0 0"/>
     <geometry>
-      <mesh filename="package://ur3robot/meshes/arm1.stl" scale="0.001 0.001 0.001"/>
+      <mesh filename="package://ur3master/meshes/arm1.stl" scale="0.001 0.001 0.001"/>
     </geometry>
     <material name="silver_default"/>
@@ -42,5 +42,5 @@
     <origin xyz="-0.143418 -0.06341 -0.829408" rpy="0 0 0"/>
     <geometry>
-      <mesh filename="package://ur3robot/meshes/arm1.stl" scale="0.001 0.001 0.001"/>
+      <mesh filename="package://ur3master/meshes/arm1.stl" scale="0.001 0.001 0.001"/>
     </geometry>
   </collision>
@@ -50,5 +50,5 @@
     <origin xyz="-0.331194 -0.06341 -0.872808" rpy="0 0 0"/>
     <geometry>
-      <mesh filename="package://ur3robot/meshes/arm2.stl" scale="0.001 0.001 0.001"/>
+      <mesh filename="package://ur3master/meshes/arm2.stl" scale="0.001 0.001 0.001"/>
     </geometry>
     <material name="silver_default"/>
@@ -57,5 +57,5 @@
     <origin xyz="-0.331194 -0.06341 -0.872808" rpy="0 0 0"/>
     <geometry>
-      <mesh filename="package://ur3robot/meshes/arm2.stl" scale="0.001 0.001 0.001"/>
+      <mesh filename="package://ur3master/meshes/arm2.stl" scale="0.001 0.001 0.001"/>
     </geometry>
   </collision>

Commit message: Updating scara code

File: ur3robot/ros_code/urdf/ur3.xacro (robot description, xacro)
@@ -137,5 +137,5 @@
 			<axis xyz="0 0 0"/>
 		</joint>
-<joint name="tower_joint" type="continuous">
+<joint name="base_link_to_tower" type="continuous">
   <origin xyz="0.105418 0.06341 0.487908" rpy="0 0 0"/>
   <parent link="base_link"/>
@@ -143,5 +143,5 @@
   <axis xyz="-0.0 0.0 -1.0"/>
 </joint>
-<joint name="arm1_joint" type="prismatic">
+<joint name="tower_to_arm1" type="prismatic">
   <origin xyz="0.038 0.0 0.3415" rpy="0 0 0"/>
   <parent link="tower"/>
@@ -150,5 +150,5 @@
   <limit upper="0.0" lower="0.0" effort="100" velocity="100"/>
 </joint>
-<joint name="arm2_joint" type="continuous">
+<joint name="arm1_to_arm2" type="continuous">
   <origin xyz="0.187776 0.0 0.0434" rpy="0 0 0"/>
   <parent link="arm1"/>

Commit message: testing

File: ur3robot/ros_code/urdf/ur3.xacro (robot description, xacro)
@@ -189,5 +189,5 @@
   <child link="arm2"/>
   <axis xyz="-0.0 -0.0 -1.0"/>
-   <limit effort="10" velocity="0.5" lower="0" upper="5.4" />
+   <limit effort="10" velocity="6.28319" lower="0" upper="5.4" />
 </joint>
 <joint name="arm2_to_end_effector" type="fixed">
