Commit message: updated urdf, and scara code

File: ur3master/ros_code/ur3master/urdf/ur3.xacro (robot description, xacro)
@@ -1,4 +1,22 @@
 <?xml version="1.0" ?>
 <robot name="ur3" xmlns:xacro="http://www.ros.org/wiki/xacro">
+<material name="blue">
+    <color rgba="0 0 0.8 1"/>
+  </material>
+  <material name="white">
+    <color rgba="1 1 1 1"/>
+  </material>
+  <material name="green">
+    <color rgba="0 0.8 0 1"/>
+  </material>
+  <material name="red">
+    <color rgba="0.8 0 0 1"/>
+  </material>
+  <material name="gray">
+    <color rgba="1 1 1 0.5"/>
+  </material>
+  <material name="black">
+    <color rgba="0 0 0 0"/>
+  </material>
 <link name="base_link">
   <visual>
@@ -7,5 +25,5 @@
       <mesh filename="package://ur3master/meshes/base_link.stl" scale="0.001 0.001 0.001"/>
     </geometry>
-    <material name="silver_default"/>
+    <material name="gray"/>
   </visual>
   <collision>
@@ -22,5 +40,5 @@
       <mesh filename="package://ur3master/meshes/tower.stl" scale="0.001 0.001 0.001"/>
     </geometry>
-    <material name="silver_default"/>
+    <material name="black"/>
   </visual>
   <collision>
@@ -37,5 +55,5 @@
       <mesh filename="package://ur3master/meshes/arm1.stl" scale="0.001 0.001 0.001"/>
     </geometry>
-    <material name="silver_default"/>
+    <material name="blue"/>
   </visual>
   <collision>
@@ -52,5 +70,5 @@
       <mesh filename="package://ur3master/meshes/arm2.stl" scale="0.001 0.001 0.001"/>
     </geometry>
-    <material name="silver_default"/>
+    <material name="green"/>
   </visual>
   <collision>
@@ -63,6 +81,4 @@
 <link name="laser">
 	</link>
-<link name="end_effector">
-  </link>
 <link name="webcam">
 	</link>
@@ -139,28 +155,24 @@
 			<axis xyz="0 0 0"/>
 		</joint>
-<joint name="base_link_to_tower" type="continuous">
+<joint name="base_link_to_tower" type="revolute">
   <origin xyz="0.105418 0.06341 0.487908" rpy="0 0 0"/>
   <parent link="base_link"/>
   <child link="tower"/>
   <axis xyz="-0.0 0.0 -1.0"/>
+  <limit effort="10" velocity="100.0" lower="-1.3708" upper="4.71239" />
 </joint>
 <joint name="tower_to_arm1" type="prismatic">
-  <origin xyz="0.038 0.0 0.3415" rpy="0 0 0"/>
+  <origin xyz="0.038 0.0 0.3415" rpy="0 0 0"/> <!-- make sure the height on this is correct-->
   <parent link="tower"/>
   <child link="arm1"/>
   <axis xyz="0.0 0.0 1.0"/>
-  <limit upper="0.0" lower="0.0" effort="100" velocity="100"/>
+  <limit upper="0.25" lower="-0.25" effort="100" velocity="100"/>
 </joint>
-<joint name="arm1_to_arm2" type="continuous">
+<joint name="arm1_to_arm2" type="revolute">
   <origin xyz="0.187776 0.0 0.0434" rpy="0 0 0"/>
   <parent link="arm1"/>
   <child link="arm2"/>
   <axis xyz="-0.0 -0.0 -1.0"/>
-</joint>
-<joint name="arm2_to_end_effector" type="fixed">
-  <origin xyz="0.187776 0.0 0" rpy="0 0 0"/>
-  <parent link="arm2"/>
-  <child link="end_effector"/>
-  <axis xyz="0.0 0.0 0"/>
+   <limit effort="10" velocity="100.0" lower="-2.7" upper="2.7" />
 </joint>
 </robot>

File: ur3robot/ros_code/urdf/ur3.xacro (robot description, xacro)
@@ -1,4 +1,22 @@
 <?xml version="1.0" ?>
 <robot name="ur3" xmlns:xacro="http://www.ros.org/wiki/xacro">
+<material name="blue">
+    <color rgba="0 0 0.8 1"/>
+  </material>
+  <material name="white">
+    <color rgba="1 1 1 1"/>
+  </material>
+  <material name="green">
+    <color rgba="0 0.8 0 1"/>
+  </material>
+  <material name="red">
+    <color rgba="0.8 0 0 1"/>
+  </material>
+  <material name="gray">
+    <color rgba="1 1 1 0.5"/>
+  </material>
+  <material name="black">
+    <color rgba="0 0 0 0"/>
+  </material>
 <link name="base_link">
   <visual>
@@ -7,5 +25,5 @@
       <mesh filename="package://ur3master/meshes/base_link.stl" scale="0.001 0.001 0.001"/>
     </geometry>
-    <material name="silver_default"/>
+    <material name="gray"/>
   </visual>
   <collision>
@@ -22,5 +40,5 @@
       <mesh filename="package://ur3master/meshes/tower.stl" scale="0.001 0.001 0.001"/>
     </geometry>
-    <material name="silver_default"/>
+    <material name="black"/>
   </visual>
   <collision>
@@ -37,5 +55,5 @@
       <mesh filename="package://ur3master/meshes/arm1.stl" scale="0.001 0.001 0.001"/>
     </geometry>
-    <material name="silver_default"/>
+    <material name="blue"/>
   </visual>
   <collision>
@@ -52,5 +70,5 @@
       <mesh filename="package://ur3master/meshes/arm2.stl" scale="0.001 0.001 0.001"/>
     </geometry>
-    <material name="silver_default"/>
+    <material name="green"/>
   </visual>
   <collision>
@@ -137,22 +155,24 @@
 			<axis xyz="0 0 0"/>
 		</joint>
-<joint name="base_link_to_tower" type="continuous">
+<joint name="base_link_to_tower" type="revolute">
   <origin xyz="0.105418 0.06341 0.487908" rpy="0 0 0"/>
   <parent link="base_link"/>
   <child link="tower"/>
   <axis xyz="-0.0 0.0 -1.0"/>
+  <limit effort="10" velocity="100.0" lower="-1.3708" upper="4.71239" />
 </joint>
 <joint name="tower_to_arm1" type="prismatic">
-  <origin xyz="0.038 0.0 0.3415" rpy="0 0 0"/>
+  <origin xyz="0.038 0.0 0.3415" rpy="0 0 0"/> <!-- make sure the height on this is correct-->
   <parent link="tower"/>
   <child link="arm1"/>
   <axis xyz="0.0 0.0 1.0"/>
-  <limit upper="0.0" lower="0.0" effort="100" velocity="100"/>
+  <limit upper="0.25" lower="-0.25" effort="100" velocity="100"/>
 </joint>
-<joint name="arm1_to_arm2" type="continuous">
+<joint name="arm1_to_arm2" type="revolute">
   <origin xyz="0.187776 0.0 0.0434" rpy="0 0 0"/>
   <parent link="arm1"/>
   <child link="arm2"/>
   <axis xyz="-0.0 -0.0 -1.0"/>
+   <limit effort="10" velocity="100.0" lower="-2.7" upper="2.7" />
 </joint>
 </robot>

Commit message: Got the moveit scara planning to do the basics!

File: ur3master/ros_code/ur3master/urdf/ur3.xacro (robot description, xacro)
@@ -76,4 +76,19 @@
     <geometry>
       <mesh filename="package://ur3master/meshes/arm2.stl" scale="0.001 0.001 0.001"/>
+    </geometry>
+  </collision>
+</link>
+<link name="end_effector">
+  <visual>
+    <origin xyz="-0.559794 -0.06341 -0.818108" rpy="0 0 0"/>
+    <geometry>
+      <mesh filename="package://ur3master/meshes/end_effector.stl" scale="0.001 0.001 0.001"/>
+    </geometry>
+    <material name="silver_default"/>
+  </visual>
+  <collision>
+    <origin xyz="-0.559794 -0.06341 -0.818108" rpy="0 0 0"/>
+    <geometry>
+      <mesh filename="package://ur3master/meshes/end_effector.stl" scale="0.001 0.001 0.001"/>
     </geometry>
   </collision>
@@ -176,3 +191,8 @@
    <limit effort="10" velocity="100.0" lower="-2.7" upper="2.7" />
 </joint>
+<joint name="arm2_to_end_effector" type="fixed">
+  <origin xyz="0.2286 0.0 -0.0547" rpy="0 0 0"/>
+  <parent link="arm2"/>
+  <child link="end_effector"/>
+</joint>
 </robot>

Commit message: working on scara

File: ur3master/ros_code/ur3master/urdf/ur3.xacro (robot description, xacro)
@@ -175,5 +175,5 @@
   <child link="tower"/>
   <axis xyz="-0.0 0.0 -1.0"/>
-  <limit effort="10" velocity="100.0" lower="-1.3708" upper="4.71239" />
+  <limit effort="10" velocity="10.0" lower="-1.0708" upper="4.71239" /> <!-- FIX ONE OFTHESE RUNS INTO LIMIT SWITCH BACK-->
 </joint>
 <joint name="tower_to_arm1" type="prismatic">
@@ -182,5 +182,5 @@
   <child link="arm1"/>
   <axis xyz="0.0 0.0 1.0"/>
-  <limit upper="0.25" lower="-0.25" effort="100" velocity="100"/>
+  <limit upper="0.25" lower="-0.25" effort="10" velocity="0.006"/>
 </joint>
 <joint name="arm1_to_arm2" type="revolute">
@@ -189,5 +189,5 @@
   <child link="arm2"/>
   <axis xyz="-0.0 -0.0 -1.0"/>
-   <limit effort="10" velocity="100.0" lower="-2.7" upper="2.7" />
+   <limit effort="10" velocity="10" lower="-2.7" upper="2.7" />
 </joint>
 <joint name="arm2_to_end_effector" type="fixed">

File: ur3robot/ros_code/urdf/ur3.xacro (robot description, xacro)
@@ -175,5 +175,5 @@
   <child link="tower"/>
   <axis xyz="-0.0 0.0 -1.0"/>
-  <limit effort="10" velocity="100.0" lower="-1.3708" upper="4.71239" />
+  <limit effort="10" velocity="100.0" lower="-1.0708" upper="4.71239" /><!-- FIX ONE OFTHESE RUNS INTO LIMIT SWITCH BACK-->
 </joint>
 <joint name="tower_to_arm1" type="prismatic">
@@ -189,5 +189,5 @@
   <child link="arm2"/>
   <axis xyz="-0.0 -0.0 -1.0"/>
-   <limit effort="10" velocity="100.0" lower="-2.7" upper="2.7" />
+   <limit effort="10" velocity="0.006" lower="-2.7" upper="2.7" />
 </joint>
 <joint name="arm2_to_end_effector" type="fixed">

Commit message: changed urdf files

File: ur3master/ros_code/ur3master/urdf/ur3.xacro (robot description, xacro)
@@ -175,5 +175,5 @@
   <child link="tower"/>
   <axis xyz="-0.0 0.0 -1.0"/>
-  <limit effort="10" velocity="10.0" lower="-1.0708" upper="4.71239" /> <!-- FIX ONE OFTHESE RUNS INTO LIMIT SWITCH BACK-->
+  <limit effort="10" velocity="2.0" lower="-1.0708" upper="4.71239" /> <!-- FIX ONE OFTHESE RUNS INTO LIMIT SWITCH BACK-->
 </joint>
 <joint name="tower_to_arm1" type="prismatic">
@@ -189,5 +189,5 @@
   <child link="arm2"/>
   <axis xyz="-0.0 -0.0 -1.0"/>
-   <limit effort="10" velocity="10" lower="-2.7" upper="2.7" />
+   <limit effort="10" velocity="2" lower="-2.7" upper="2.7" />
 </joint>
 <joint name="arm2_to_end_effector" type="fixed">

File: ur3robot/ros_code/urdf/ur3.xacro (robot description, xacro)
@@ -175,5 +175,5 @@
   <child link="tower"/>
   <axis xyz="-0.0 0.0 -1.0"/>
-  <limit effort="10" velocity="100.0" lower="-1.0708" upper="4.71239" /><!-- FIX ONE OFTHESE RUNS INTO LIMIT SWITCH BACK-->
+  <limit effort="10" velocity="2.0" lower="-1.0708" upper="4.71239" /><!-- FIX ONE OFTHESE RUNS INTO LIMIT SWITCH BACK-->
 </joint>
 <joint name="tower_to_arm1" type="prismatic">
@@ -182,5 +182,5 @@
   <child link="arm1"/>
   <axis xyz="0.0 0.0 1.0"/>
-  <limit upper="0.25" lower="-0.25" effort="100" velocity="100"/>
+  <limit upper="0.25" lower="-0.25" effort="100" velocity="0.006"/>
 </joint>
 <joint name="arm1_to_arm2" type="revolute">
@@ -189,5 +189,5 @@
   <child link="arm2"/>
   <axis xyz="-0.0 -0.0 -1.0"/>
-   <limit effort="10" velocity="0.006" lower="-2.7" upper="2.7" />
+   <limit effort="10" velocity="2" lower="-2.7" upper="2.7" />
 </joint>
 <joint name="arm2_to_end_effector" type="fixed">
