Commit message: Updated robots urdf to include the new camera and bottle pickerupper.

File: ur3master/ros_code/ur3master/urdf/ur3.xacro (robot description, xacro)
@@ -38,5 +38,5 @@
     <origin xyz="-0.105418 -0.06341 -0.486908" rpy="0 0 0"/>
     <geometry>
-      <mesh filename="package://ur3master/meshes/tower.stl" scale="0.001 0.001 0.001"/>
+      <mesh filename="package://ur3_description/meshes/tower.stl" scale="0.001 0.001 0.001"/>
     </geometry>
     <material name="black"/>
@@ -45,5 +45,5 @@
     <origin xyz="-0.105418 -0.06341 -0.486908" rpy="0 0 0"/>
     <geometry>
-      <mesh filename="package://ur3master/meshes/tower.stl" scale="0.001 0.001 0.001"/>
+      <mesh filename="package://ur3_description/meshes/tower.stl" scale="0.001 0.001 0.001"/>
     </geometry>
   </collision>
@@ -53,5 +53,5 @@
     <origin xyz="-0.067418 -0.06341 -0.6118" rpy="0 0 0"/>
     <geometry>
-      <mesh filename="package://ur3master/meshes/arm1.stl" scale="0.001 0.001 0.001"/>
+      <mesh filename="package://ur3_description/meshes/arm1.stl" scale="0.001 0.001 0.001"/>
     </geometry>
     <material name="blue"/>
@@ -60,5 +60,35 @@
     <origin xyz="-0.067418 -0.06341 -0.6118" rpy="0 0 0"/>
     <geometry>
-      <mesh filename="package://ur3master/meshes/arm1.stl" scale="0.001 0.001 0.001"/>
+      <mesh filename="package://ur3_description/meshes/arm1.stl" scale="0.001 0.001 0.001"/>
+    </geometry>
+  </collision>
+</link>
+<link name="arm_camera">
+  <visual>
+    <origin xyz="0.348957 -0.06341 -0.6205" rpy="0 0 0"/>
+    <geometry>
+      <mesh filename="package://ur3_description/meshes/arm_camera.stl" scale="0.001 0.001 0.001"/>
+    </geometry>
+    <material name="silver_default"/>
+  </visual>
+  <collision>
+    <origin xyz="0.348957 -0.06341 -0.6205" rpy="0 0 0"/>
+    <geometry>
+      <mesh filename="package://ur3_description/meshes/arm_camera.stl" scale="0.001 0.001 0.001"/>
+    </geometry>
+  </collision>
+</link>
+<link name="end_effector">
+  <visual>
+    <origin xyz="0.315207 -0.06341 -0.6005" rpy="0 0 0"/>
+    <geometry>
+      <mesh filename="package://ur3_description/meshes/end_effector.stl" scale="0.001 0.001 0.001"/>
+    </geometry>
+    <material name="silver_default"/>
+  </visual>
+  <collision>
+    <origin xyz="0.315207 -0.06341 -0.6005" rpy="0 0 0"/>
+    <geometry>
+      <mesh filename="package://ur3_description/meshes/end_effector.stl" scale="0.001 0.001 0.001"/>
     </geometry>
   </collision>
@@ -68,5 +98,5 @@
     <origin xyz="0.120357 -0.06341 -0.6552" rpy="0 0 0"/>
     <geometry>
-      <mesh filename="package://ur3master/meshes/arm2.stl" scale="0.001 0.001 0.001"/>
+      <mesh filename="package://ur3_description/meshes/arm2.stl" scale="0.001 0.001 0.001"/>
     </geometry>
     <material name="green"/>
@@ -75,20 +105,5 @@
     <origin xyz="0.120357 -0.06341 -0.6552" rpy="0 0 0"/>
     <geometry>
-      <mesh filename="package://ur3master/meshes/arm2.stl" scale="0.001 0.001 0.001"/>
-    </geometry>
-  </collision>
-</link>
-<link name="end_effector">
-  <visual>
-    <origin xyz="-0.086312 0.034291 -0.6005" rpy="0 0 0"/>
-    <geometry>
-      <mesh filename="package://ur3master/meshes/end_effector.stl" scale="0.001 0.001 0.001"/>
-    </geometry>
-    <material name="silver_default"/>
-  </visual>
-  <collision>
-    <origin xyz="-0.086312 0.034291 -0.6005" rpy="0 0 0"/>
-    <geometry>
-      <mesh filename="package://ur3master/meshes/end_effector.stl" scale="0.001 0.001 0.001"/>
+      <mesh filename="package://ur3_description/meshes/arm2.stl" scale="0.001 0.001 0.001"/>
     </geometry>
   </collision>
@@ -174,5 +189,5 @@
   <parent link="base_link"/>
   <child link="tower"/>
-  <axis xyz="-0.0 0.0 -1.0"/>
+  <axis xyz="0.0 -0.0 1.0"/>
   <limit effort="10" velocity="0.75" lower="-4.21239" upper="1.59534" /><!-- Set lower to proper value to prevent tower hitting limit switch-->
 </joint>
@@ -184,15 +199,20 @@
   <limit upper="0.5" lower="0.0" effort="10" velocity="0.006"/> <!-- make sure that the arm can actually go up 0.5-->
 </joint>
+<joint name="arm2_to_camera" type="fixed">
+  <origin xyz="-0.2286 0.0 -0.0347" rpy="0 0 0"/>
+  <parent link="arm2"/>
+  <child link="camera"/>
+</joint>
+<joint name="arm2_to_end_effector" type="fixed">
+  <origin xyz="-0.19485 0.0 -0.0547" rpy="0 0 0"/>
+  <parent link="arm2"/>
+  <child link="end_effector"/>
+</joint>
 <joint name="arm1_to_arm2" type="revolute">
   <origin xyz="-0.187775 0.0 0.0434" rpy="0 0 0"/>
   <parent link="arm1"/>
   <child link="arm2"/>
-  <axis xyz="-0.0 -0.0 -1.0"/>
-   <limit effort="10" velocity="0.31415" lower="0" upper="5.4" />
-</joint>
-<joint name="arm2_to_end_effector" type="fixed">
-  <origin xyz="0.206669 -0.097701 -0.0547" rpy="0 0 0"/>
-  <parent link="arm2"/>
-  <child link="end_effector"/>
+  <axis xyz="0.0 0.0 -1.0"/>
+  <limit effort="10" velocity="0.31415" lower="0" upper="5.4" /> <!-- fix the bounderies -->
 </joint>
 </robot>

Commit message: fixed urdf

File: ur3master/ros_code/ur3master/urdf/ur3.xacro (robot description, xacro)
@@ -199,8 +199,8 @@
   <limit upper="0.5" lower="0.0" effort="10" velocity="0.006"/> <!-- make sure that the arm can actually go up 0.5-->
 </joint>
-<joint name="arm2_to_camera" type="fixed">
+<joint name="arm2_to_arm_camera" type="fixed">
   <origin xyz="-0.2286 0.0 -0.0347" rpy="0 0 0"/>
   <parent link="arm2"/>
-  <child link="camera"/>
+  <child link="arm_camera"/>
 </joint>
 <joint name="arm2_to_end_effector" type="fixed">

Commit message: updated scara config, working on urdf

File: ur3master/ros_code/ur3master/urdf/ur3.xacro (robot description, xacro)
@@ -38,5 +38,5 @@
     <origin xyz="-0.105418 -0.06341 -0.486908" rpy="0 0 0"/>
     <geometry>
-      <mesh filename="package://ur3_description/meshes/tower.stl" scale="0.001 0.001 0.001"/>
+      <mesh filename="package://ur3master/meshes/tower.stl" scale="0.001 0.001 0.001"/>
     </geometry>
     <material name="black"/>
@@ -45,5 +45,5 @@
     <origin xyz="-0.105418 -0.06341 -0.486908" rpy="0 0 0"/>
     <geometry>
-      <mesh filename="package://ur3_description/meshes/tower.stl" scale="0.001 0.001 0.001"/>
+      <mesh filename="package://ur3master/meshes/tower.stl" scale="0.001 0.001 0.001"/>
     </geometry>
   </collision>
@@ -53,5 +53,5 @@
     <origin xyz="-0.067418 -0.06341 -0.6118" rpy="0 0 0"/>
     <geometry>
-      <mesh filename="package://ur3_description/meshes/arm1.stl" scale="0.001 0.001 0.001"/>
+      <mesh filename="package://ur3master/meshes/arm1.stl" scale="0.001 0.001 0.001"/>
     </geometry>
     <material name="blue"/>
@@ -60,5 +60,5 @@
     <origin xyz="-0.067418 -0.06341 -0.6118" rpy="0 0 0"/>
     <geometry>
-      <mesh filename="package://ur3_description/meshes/arm1.stl" scale="0.001 0.001 0.001"/>
+      <mesh filename="package://ur3master/meshes/arm1.stl" scale="0.001 0.001 0.001"/>
     </geometry>
   </collision>
@@ -68,5 +68,5 @@
     <origin xyz="0.348957 -0.06341 -0.6205" rpy="0 0 0"/>
     <geometry>
-      <mesh filename="package://ur3_description/meshes/arm_camera.stl" scale="0.001 0.001 0.001"/>
+      <mesh filename="package://ur3master/meshes/arm_camera.stl" scale="0.001 0.001 0.001"/>
     </geometry>
     <material name="silver_default"/>
@@ -75,5 +75,5 @@
     <origin xyz="0.348957 -0.06341 -0.6205" rpy="0 0 0"/>
     <geometry>
-      <mesh filename="package://ur3_description/meshes/arm_camera.stl" scale="0.001 0.001 0.001"/>
+      <mesh filename="package://ur3master/meshes/arm_camera.stl" scale="0.001 0.001 0.001"/>
     </geometry>
   </collision>
@@ -83,5 +83,5 @@
     <origin xyz="0.315207 -0.06341 -0.6005" rpy="0 0 0"/>
     <geometry>
-      <mesh filename="package://ur3_description/meshes/end_effector.stl" scale="0.001 0.001 0.001"/>
+      <mesh filename="package://ur3master/meshes/end_effector.stl" scale="0.001 0.001 0.001"/>
     </geometry>
     <material name="silver_default"/>
@@ -90,5 +90,5 @@
     <origin xyz="0.315207 -0.06341 -0.6005" rpy="0 0 0"/>
     <geometry>
-      <mesh filename="package://ur3_description/meshes/end_effector.stl" scale="0.001 0.001 0.001"/>
+      <mesh filename="package://ur3master/meshes/end_effector.stl" scale="0.001 0.001 0.001"/>
     </geometry>
   </collision>
@@ -98,5 +98,5 @@
     <origin xyz="0.120357 -0.06341 -0.6552" rpy="0 0 0"/>
     <geometry>
-      <mesh filename="package://ur3_description/meshes/arm2.stl" scale="0.001 0.001 0.001"/>
+      <mesh filename="package://ur3master/meshes/arm2.stl" scale="0.001 0.001 0.001"/>
     </geometry>
     <material name="green"/>
@@ -105,5 +105,5 @@
     <origin xyz="0.120357 -0.06341 -0.6552" rpy="0 0 0"/>
     <geometry>
-      <mesh filename="package://ur3_description/meshes/arm2.stl" scale="0.001 0.001 0.001"/>
+      <mesh filename="package://ur3master/meshes/arm2.stl" scale="0.001 0.001 0.001"/>
     </geometry>
   </collision>
@@ -189,6 +189,6 @@
   <parent link="base_link"/>
   <child link="tower"/>
-  <axis xyz="0.0 -0.0 1.0"/>
-  <limit effort="10" velocity="0.75" lower="-4.21239" upper="1.59534" /><!-- Set lower to proper value to prevent tower hitting limit switch-->
+  <axis xyz="0.0 0.0 -1.0"/>
+  <limit effort="10" velocity="0.75" lower="-1.59534" upper="4.21239" /><!-- Set lower to proper value to prevent tower hitting limit switch-->
 </joint>
 <joint name="tower_to_arm1" type="prismatic">
@@ -214,5 +214,5 @@
   <child link="arm2"/>
   <axis xyz="0.0 0.0 -1.0"/>
-  <limit effort="10" velocity="0.31415" lower="0" upper="5.4" /> <!-- fix the bounderies -->
+  <limit effort="10" velocity="0.31415" lower="-2.6" upper="2.4" /> <!-- fix the bounderies -->
 </joint>
 </robot>

File: ur3robot/ros_code/urdf/ur3.xacro (robot description, xacro)
@@ -30,5 +30,5 @@
     <origin xyz="0 0 0" rpy="0 0 0"/>
     <geometry>
-      <mesh filename="package://ur3master/meshes/base_link.stl" scale="0.001 0.001 0.001"/>
+      <mesh filename="package://ur3robot/meshes/base_link.stl" scale="0.001 0.001 0.001"/>
     </geometry>
   </collision>
@@ -38,5 +38,5 @@
     <origin xyz="-0.105418 -0.06341 -0.486908" rpy="0 0 0"/>
     <geometry>
-      <mesh filename="package://ur3_description/meshes/tower.stl" scale="0.001 0.001 0.001"/>
+      <mesh filename="package://ur3robot/meshes/tower.stl" scale="0.001 0.001 0.001"/>
     </geometry>
     <material name="black"/>
@@ -45,5 +45,5 @@
     <origin xyz="-0.105418 -0.06341 -0.486908" rpy="0 0 0"/>
     <geometry>
-      <mesh filename="package://ur3_description/meshes/tower.stl" scale="0.001 0.001 0.001"/>
+      <mesh filename="package://ur3robot/meshes/tower.stl" scale="0.001 0.001 0.001"/>
     </geometry>
   </collision>
@@ -53,5 +53,5 @@
     <origin xyz="-0.067418 -0.06341 -0.6118" rpy="0 0 0"/>
     <geometry>
-      <mesh filename="package://ur3_description/meshes/arm1.stl" scale="0.001 0.001 0.001"/>
+      <mesh filename="package://ur3robot/meshes/arm1.stl" scale="0.001 0.001 0.001"/>
     </geometry>
     <material name="blue"/>
@@ -60,5 +60,5 @@
     <origin xyz="-0.067418 -0.06341 -0.6118" rpy="0 0 0"/>
     <geometry>
-      <mesh filename="package://ur3_description/meshes/arm1.stl" scale="0.001 0.001 0.001"/>
+      <mesh filename="package://ur3robot/meshes/arm1.stl" scale="0.001 0.001 0.001"/>
     </geometry>
   </collision>
@@ -68,5 +68,5 @@
     <origin xyz="0.348957 -0.06341 -0.6205" rpy="0 0 0"/>
     <geometry>
-      <mesh filename="package://ur3_description/meshes/arm_camera.stl" scale="0.001 0.001 0.001"/>
+      <mesh filename="package://ur3robot/meshes/arm_camera.stl" scale="0.001 0.001 0.001"/>
     </geometry>
     <material name="silver_default"/>
@@ -75,5 +75,5 @@
     <origin xyz="0.348957 -0.06341 -0.6205" rpy="0 0 0"/>
     <geometry>
-      <mesh filename="package://ur3_description/meshes/arm_camera.stl" scale="0.001 0.001 0.001"/>
+      <mesh filename="package://ur3robot/meshes/arm_camera.stl" scale="0.001 0.001 0.001"/>
     </geometry>
   </collision>
@@ -83,5 +83,5 @@
     <origin xyz="0.315207 -0.06341 -0.6005" rpy="0 0 0"/>
     <geometry>
-      <mesh filename="package://ur3_description/meshes/end_effector.stl" scale="0.001 0.001 0.001"/>
+      <mesh filename="package://ur3robot/meshes/end_effector.stl" scale="0.001 0.001 0.001"/>
     </geometry>
     <material name="silver_default"/>
@@ -90,5 +90,5 @@
     <origin xyz="0.315207 -0.06341 -0.6005" rpy="0 0 0"/>
     <geometry>
-      <mesh filename="package://ur3_description/meshes/end_effector.stl" scale="0.001 0.001 0.001"/>
+      <mesh filename="package://ur3robot/meshes/end_effector.stl" scale="0.001 0.001 0.001"/>
     </geometry>
   </collision>
@@ -98,5 +98,5 @@
     <origin xyz="0.120357 -0.06341 -0.6552" rpy="0 0 0"/>
     <geometry>
-      <mesh filename="package://ur3_description/meshes/arm2.stl" scale="0.001 0.001 0.001"/>
+      <mesh filename="package://ur3robot/meshes/arm2.stl" scale="0.001 0.001 0.001"/>
     </geometry>
     <material name="green"/>
@@ -105,5 +105,5 @@
     <origin xyz="0.120357 -0.06341 -0.6552" rpy="0 0 0"/>
     <geometry>
-      <mesh filename="package://ur3_description/meshes/arm2.stl" scale="0.001 0.001 0.001"/>
+      <mesh filename="package://ur3robot/meshes/arm2.stl" scale="0.001 0.001 0.001"/>
     </geometry>
   </collision>
@@ -189,6 +189,6 @@
   <parent link="base_link"/>
   <child link="tower"/>
-  <axis xyz="0.0 -0.0 1.0"/>
-  <limit effort="10" velocity="0.75" lower="-4.21239" upper="1.59534" /><!-- Set lower to proper value to prevent tower hitting limit switch-->
+  <axis xyz="0.0 0.0 -1.0"/>
+  <limit effort="10" velocity="0.75" lower="-1.59534" upper="4.21239" /><!-- Set lower to proper value to prevent tower hitting limit switch-->
 </joint>
 <joint name="tower_to_arm1" type="prismatic">
@@ -214,5 +214,5 @@
   <child link="arm2"/>
   <axis xyz="0.0 0.0 -1.0"/>
-  <limit effort="10" velocity="0.31415" lower="0" upper="5.4" /> <!-- fix the bounderies -->
+  <limit effort="10" velocity="0.31415" lower="-2.6" upper="2.4" /> <!-- fix the bounderies -->
 </joint>
 </robot>

Commit message: fixed some xacro file stuff

File: ur3master/ros_code/ur3master/urdf/ur3.xacro (robot description, xacro)
@@ -190,5 +190,5 @@
   <child link="tower"/>
   <axis xyz="0.0 0.0 -1.0"/>
-  <limit effort="10" velocity="0.75" lower="-1.59534" upper="4.21239" /><!-- Set lower to proper value to prevent tower hitting limit switch-->
+  <limit effort="10" velocity="0.75" lower="-4.21239" upper="1.59534" /><!-- Set lower to proper value to prevent tower hitting limit switch-->
 </joint>
 <joint name="tower_to_arm1" type="prismatic">

File: ur3robot/ros_code/urdf/ur3.xacro (robot description, xacro)
@@ -190,5 +190,5 @@
   <child link="tower"/>
   <axis xyz="0.0 0.0 -1.0"/>
-  <limit effort="10" velocity="0.75" lower="-1.59534" upper="4.21239" /><!-- Set lower to proper value to prevent tower hitting limit switch-->
+  <limit effort="10" velocity="0.75" lower="-4.21239" upper="1.59534" /><!-- Set lower to proper value to prevent tower hitting limit switch-->
 </joint>
 <joint name="tower_to_arm1" type="prismatic">
